File: Stepper Motor Prototype.sch (KiCad schematic (older format))
At the start: 45 parts, among them J1 USB_B_Micro, J2 Screw_Terminal_01x02, J3 Screw_Terminal_01x04, Q1 STD20NF06L, Q2 STD20NF06L, Q3 STD20NF06L, Q4 STD20NF06L, Q5 STD20NF06L, Q6 STD20NF06L, Q7 STD20NF06L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

Commit message: committing before ripping whole board up.  Board will now only contain power seciton and 1 stepper driver
Parts:
- removed U4: MSP430G2553IPW28, Housings_SSOP:TSSOP-28_4.4x9.7mm_Pitch0.65mm, symbol MCU_Texas_MSP430:MSP430G2553IPW28
- added C11, C13: 120uF, Capacitors_THT:CP_Radial_D8.0mm_P3.50mm, symbol Device:C
- added C15, C16: C, Capacitors_SMD:C_0603_HandSoldering, symbol Device:C
- added C17, C18, C19, C20, C21, C22, C23, C24: 0.1uF, Capacitors_SMD:C_0603_HandSoldering, symbol Device:C
- added R7, R8: 0.05R, Resistors_SMD:R_2512, symbol Device:R
- added TP1, TP2, TP3, TP4: TestPoint, Measurement_Points:Test_Point_Keystone_5010-5014_Multipurpose, symbol Connector:TestPoint
- added U8: STM32F407VGTx, Housings_QFP:LQFP-100_14x14mm_Pitch0.5mm, symbol MCU_ST_STM32F4:STM32F407VGTx
- added Y1: Crystal_GND24, Crystals:Crystal_SMD_SeikoEpson_TSX3225-4pin_3.2x2.5mm, symbol Device:Crystal_GND24
- C1: footprint Capacitors_SMD:C_0603_HandSoldering -> Capacitors_THT:CP_Radial_D8.0mm_P3.50mm
- C12, C14: renamed from C?; value 4.7uF -> 150uF; footprint Capacitors_SMD:C_0603_HandSoldering -> Capacitors_THT:CP_Radial_D8.0mm_P3.50mm
- D4: renamed from D?; footprint (none) -> digikey-footprints:DO-214AB; Vishay P/N (none) -> MURS320-E3/57T
- D6: renamed from D?; footprint (none) -> digikey-footprints:DO-214AB
- L1, L2: renamed from L?; footprint (none) -> my_inductors:Wurth_SMD_Inductor_7447709101
- U7: footprint Housings_SSOP:TSSOP-38_4.4x9.7mm_Pitch0.5mm -> rca_switch_through_hole:TSSOP-38-1_PowerPad_4.4x9.7mm_Pitch0.5mm
- gave numbers to parts that had none: 4
Connections:
- net labels added: FTDI_BYPASS, ST_P100, ST_P11, ST_P19, ST_P22, ST_P28, ST_P50, ST_P6, ST_P75
- wire segments 76 -> 208
